Commit message: modified the official urdf file to be able to locate those meshes

File: ubt_sim_ws/src/example/config/walker.urdf (robot description, URDF)
Before this commit: robot walker_description, 56 links, 55 joints
Links:
- link base_link: geometry collision mesh filename=package://example/meshes/base_link.STL; visual mesh filename=package://example/meshes/base_link.STL
- link head_l1: geometry collision mesh filename=package://example/meshes/head_l1.STL; visual mesh filename=package://example/meshes/head_l1.STL
- link head_l2: geometry collision mesh filename=package://example/meshes/head_l2.STL; visual mesh filename=package://example/meshes/head_l2.STL
- link head_l3: geometry collision mesh filename=package://example/meshes/head_l3.STL; visual mesh filename=package://example/meshes/head_l3.STL
- link left_index_l1: geometry collision mesh filename=package://example/meshes/left_index_l1.STL; visual mesh filename=package://example/meshes/left_index_l1.STL
- link left_index_l2: geometry collision mesh filename=package://example/meshes/left_index_l2.STL; visual mesh filename=package://example/meshes/left_index_l2.STL
- link left_leg_l1: geometry collision mesh filename=package://example/meshes/left_leg_l1.STL; visual mesh filename=package://example/meshes/left_leg_l1.STL
- link left_leg_l2: geometry collision mesh filename=package://example/meshes/left_leg_l2.STL; visual mesh filename=package://example/meshes/left_leg_l2.STL
- link left_leg_l3: geometry collision mesh filename=package://example/meshes/left_leg_l3.STL; visual mesh filename=package://example/meshes/left_leg_l3.STL
- link left_leg_l4: geometry collision mesh filename=package://example/meshes/left_leg_l4.STL; visual mesh filename=package://example/meshes/left_leg_l4.STL
- link left_leg_l5: geometry collision mesh filename=package://example/meshes/left_leg_l5.STL; visual mesh filename=package://example/meshes/left_leg_l5.STL
- link left_leg_l6: geometry collision mesh filename=package://example/meshes/left_leg_l6.STL; visual mesh filename=package://example/meshes/left_leg_l6.STL
- link left_leg_link1: geometry collision mesh filename=package://example/meshes/left_leg_link1.STL; visual mesh filename=package://example/meshes/left_leg_link1.STL
- link left_leg_link2: geometry collision mesh filename=package://example/meshes/left_leg_link2.STL; visual mesh filename=package://example/meshes/left_leg_link2.STL
- link left_limb_l1: geometry collision mesh filename=package://example/meshes/left_limb_l1.STL; visual mesh filename=package://example/meshes/left_limb_l1.STL
- link left_limb_l2: geometry collision mesh filename=package://example/meshes/left_limb_l2.STL; visual mesh filename=package://example/meshes/left_limb_l2.STL
- link left_limb_l3: geometry collision mesh filename=package://example/meshes/left_limb_l3.STL; visual mesh filename=package://example/meshes/left_limb_l3.STL
- link left_limb_l4: geometry collision mesh filename=package://example/meshes/left_limb_l4.STL; visual mesh filename=package://example/meshes/left_limb_l4.STL
- link left_limb_l5: geometry collision mesh filename=package://example/meshes/left_limb_l5.STL; visual mesh filename=package://example/meshes/left_limb_l5.STL
- link left_limb_l6: geometry collision mesh filename=package://example/meshes/left_limb_l6.STL; visual mesh filename=package://example/meshes/left_limb_l6.STL
- link left_limb_l7: geometry collision mesh filename=package://example/meshes/left_limb_l7.STL; visual mesh filename=package://example/meshes/left_limb_l7.STL
- link left_middle_l1: geometry collision mesh filename=package://example/meshes/left_middle_l1.STL; visual mesh filename=package://example/meshes/left_middle_l1.STL
- link left_middle_l2: geometry collision mesh filename=package://example/meshes/left_middle_l2.STL; visual mesh filename=package://example/meshes/left_middle_l2.STL
- link left_palm_link: geometry collision mesh filename=package://example/meshes/left_palm_link.STL; visual mesh filename=package://example/meshes/left_palm_link.STL
- link left_pinky_l1: geometry collision mesh filename=package://example/meshes/left_pinky_l1.STL; visual mesh filename=package://example/meshes/left_pinky_l1.STL
- link left_pinky_l2: geometry collision mesh filename=package://example/meshes/left_pinky_l2.STL; visual mesh filename=package://example/meshes/left_pinky_l2.STL
- link left_ring_l1: geometry collision mesh filename=package://example/meshes/left_ring_l1.STL; visual mesh filename=package://example/meshes/left_ring_l1.STL
- link left_ring_l2: geometry collision mesh filename=package://example/meshes/left_ring_l2.STL; visual mesh filename=package://example/meshes/left_ring_l2.STL
- link left_thumb_l1: geometry collision mesh filename=package://example/meshes/left_thumb_l1.STL; visual mesh filename=package://example/meshes/left_thumb_l1.STL
- link left_thumb_l2: geometry collision mesh filename=package://example/meshes/left_thumb_l2.STL; visual mesh filename=package://example/meshes/left_thumb_l2.STL
- link right_index_l1: geometry collision mesh filename=package://example/meshes/right_index_l1.STL; visual mesh filename=package://example/meshes/right_index_l1.STL
- link right_index_l2: geometry collision mesh filename=package://example/meshes/right_index_l2.STL; visual mesh filename=package://example/meshes/right_index_l2.STL
- link right_leg_l1: geometry collision mesh filename=package://example/meshes/right_leg_l1.STL; visual mesh filename=package://example/meshes/right_leg_l1.STL
- link right_leg_l2: geometry collision mesh filename=package://example/meshes/right_leg_l2.STL; visual mesh filename=package://example/meshes/right_leg_l2.STL
- link right_leg_l3: geometry collision mesh filename=package://example/meshes/right_leg_l3.STL; visual mesh filename=package://example/meshes/right_leg_l3.STL
- link right_leg_l4: geometry collision mesh filename=package://example/meshes/right_leg_l4.STL; visual mesh filename=package://example/meshes/right_leg_l4.STL
- link right_leg_l5: geometry collision mesh filename=package://example/meshes/right_leg_l5.STL; visual mesh filename=package://example/meshes/right_leg_l5.STL
- link right_leg_l6: geometry collision mesh filename=package://example/meshes/right_leg_l6.STL; visual mesh filename=package://example/meshes/right_leg_l6.STL
- link right_leg_link1: geometry collision mesh filename=package://example/meshes/right_leg_link1.STL; visual mesh filename=package://example/meshes/right_leg_link1.STL
- link right_leg_link2: geometry collision mesh filename=package://example/meshes/right_leg_link2.STL; visual mesh filename=package://example/meshes/right_leg_link2.STL
- link right_limb_l1: geometry collision mesh filename=package://example/meshes/right_limb_l1.STL; visual mesh filename=package://example/meshes/right_limb_l1.STL
- link right_limb_l2: geometry collision mesh filename=package://example/meshes/right_limb_l2.STL; visual mesh filename=package://example/meshes/right_limb_l2.STL
- link right_limb_l3: geometry collision mesh filename=package://example/meshes/right_limb_l3.STL; visual mesh filename=package://example/meshes/right_limb_l3.STL
- link right_limb_l4: geometry collision mesh filename=package://example/meshes/right_limb_l4.STL; visual mesh filename=package://example/meshes/right_limb_l4.STL
- link right_limb_l5: geometry collision mesh filename=package://example/meshes/right_limb_l5.STL; visual mesh filename=package://example/meshes/right_limb_l5.STL
- link right_limb_l6: geometry collision mesh filename=package://example/meshes/right_limb_l6.STL; visual mesh filename=package://example/meshes/right_limb_l6.STL
- link right_limb_l7: geometry collision mesh filename=package://example/meshes/right_limb_l7.STL; visual mesh filename=package://example/meshes/right_limb_l7.STL
- link right_middle_l1: geometry collision mesh filename=package://example/meshes/right_middle_l1.STL; visual mesh filename=package://example/meshes/right_middle_l1.STL
- link right_middle_l2: geometry collision mesh filename=package://example/meshes/right_middle_l2.STL; visual mesh filename=package://example/meshes/right_middle_l2.STL
- link right_palm_link: geometry collision mesh filename=package://example/meshes/right_palm_link.STL; visual mesh filename=package://example/meshes/right_palm_link.STL
- link right_pinky_l1: geometry collision mesh filename=package://example/meshes/right_pinky_l1.STL; visual mesh filename=package://example/meshes/right_pinky_l1.STL
- link right_pinky_l2: geometry collision mesh filename=package://example/meshes/right_pinky_l2.STL; visual mesh filename=package://example/meshes/right_pinky_l2.STL
- link right_ring_l1: geometry collision mesh filename=package://example/meshes/right_ring_l1.STL; visual mesh filename=package://example/meshes/right_ring_l1.STL
- link right_ring_l2: geometry collision mesh filename=package://example/meshes/right_ring_l2.STL; visual mesh filename=package://example/meshes/right_ring_l2.STL
- link right_thumb_l1: geometry collision mesh filename=package://example/meshes/right_thumb_l1.STL; visual mesh filename=package://example/meshes/right_thumb_l1.STL
- link right_thumb_l2: geometry collision mesh filename=package://example/meshes/right_thumb_l2.STL; visual mesh filename=package://example/meshes/right_thumb_l2.STL
