Commit message: add effort to new urdf, the others are not changed

File: ubt_sim_ws/src/walker_description/urdf/walker_webots.urdf (robot description, URDF)
Before this commit: robot walker, 56 links, 55 joints
Joints:
- joint head_j1: limit lower=-1.6572 upper=1.6572 effort=0 velocity=0 -> lower=-1.6572 upper=1.6572 effort=3.5 velocity=0
- joint head_j2: limit lower=-0.5232 upper=0.5232 effort=0 velocity=0 -> lower=-0.5232 upper=0.5232 effort=3.5 velocity=0
- joint left_leg_j1: limit lower=-0.8722 upper=0.8722 effort=0 velocity=0 -> lower=-0.8722 upper=0.8722 effort=160 velocity=0
- joint left_leg_j2: limit lower=-0.6112 upper=0.6112 effort=0 velocity=0 -> lower=-0.6112 upper=0.6112 effort=270 velocity=0
- joint left_leg_j3: limit lower=-1.4872 upper=0.6112 effort=0 velocity=0 -> lower=-1.4872 upper=0.6112 effort=270 velocity=0
- joint left_leg_j4: limit lower=-0.2622 upper=2.2672 effort=0 velocity=0 -> lower=-0.2622 upper=2.2672 effort=270 velocity=0
- joint left_leg_j5: limit lower=-1.4872 upper=0.6112 effort=0 velocity=0 -> lower=-1.4872 upper=0.6112 effort=160 velocity=0
- joint left_leg_j6: limit lower=-0.6112 upper=0.6112 effort=0 velocity=0 -> lower=-0.6112 upper=0.6112 effort=160 velocity=0
- joint left_limb_j1: limit lower=-0.8722 upper=3.1416 effort=0 velocity=0 -> lower=-0.8722 upper=3.1416 effort=96.2 velocity=0
- joint left_limb_j2: limit lower=-1.6572 upper=0.1047 effort=0 velocity=0 -> lower=-1.6572 upper=0.1047 effort=96.2 velocity=0
- joint left_limb_j3: limit lower=-2.0072 upper=2.0072 effort=0 velocity=0 -> lower=-2.0072 upper=2.0072 effort=96.2 velocity=0
- joint left_limb_j4: limit lower=-2.3572 upper=0 effort=0 velocity=0 -> lower=-2.3572 upper=0 effort=96.2 velocity=0
- joint left_limb_j5: limit lower=-2.4472 upper=2.4472 effort=0 velocity=0 -> lower=-2.4472 upper=2.4472 effort=27.3 velocity=0
- joint left_limb_j6: limit lower=-0.8722 upper=0.8722 effort=0 velocity=0 -> lower=-0.8722 upper=0.8722 effort=27.3 velocity=0
- joint left_limb_j7: limit lower=-0.8722 upper=0.8722 effort=0 velocity=0 -> lower=-0.8722 upper=0.8722 effort=27.3 velocity=0
- joint right_leg_j1: limit lower=-0.8722 upper=0.8722 effort=0 velocity=0 -> lower=-0.8722 upper=0.8722 effort=160 velocity=0
- joint right_leg_j2: limit lower=-0.6112 upper=0.6112 effort=0 velocity=0 -> lower=-0.6112 upper=0.6112 effort=270 velocity=0
- joint right_leg_j3: limit lower=-1.4872 upper=0.6112 effort=0 velocity=0 -> lower=-1.4872 upper=0.6112 effort=270 velocity=0
- joint right_leg_j4: limit lower=-0.2622 upper=2.2672 effort=0 velocity=0 -> lower=-0.2622 upper=2.2672 effort=270 velocity=0
- joint right_leg_j5: limit lower=-1.4872 upper=0.6112 effort=0 velocity=0 -> lower=-1.4872 upper=0.6112 effort=160 velocity=0
- joint right_leg_j6: limit lower=-0.6112 upper=0.6112 effort=0 velocity=0 -> lower=-0.6112 upper=0.6112 effort=160 velocity=0
- joint right_limb_j1: limit lower=-3.1416 upper=0.8722 effort=0 velocity=0 -> lower=-3.1416 upper=0.8722 effort=96.2 velocity=0
- joint right_limb_j2: limit lower=-1.6572 upper=0.1047 effort=0 velocity=0 -> lower=-1.6572 upper=0.1047 effort=96.2 velocity=0
- joint right_limb_j3: limit lower=-2.0072 upper=2.0072 effort=0 velocity=0 -> lower=-2.0072 upper=2.0072 effort=96.2 velocity=0
- joint right_limb_j4: limit lower=-2.3572 upper=0 effort=0 velocity=0 -> lower=-2.3572 upper=0 effort=27.3 velocity=0
- joint right_limb_j5: limit lower=-2.4472 upper=2.4472 effort=0 velocity=0 -> lower=-2.4472 upper=2.4472 effort=27.3 velocity=0
- joint right_limb_j6: limit lower=-0.8722 upper=0.8722 effort=0 velocity=0 -> lower=-0.8722 upper=0.8722 effort=27.3 velocity=0
- joint right_limb_j7: limit lower=-0.8722 upper=0.8722 effort=0 velocity=0 -> lower=-0.8722 upper=0.8722 effort=0.5 velocity=0
