Commit message: fixed namespace issue in moveit.launch

File: ubt_sim_ws/src/walker_description/urdf/walker.urdf (robot description, URDF)
Before this commit: robot walker, 56 links, 55 joints
Links:
- link head_l1: geometry 
- link head_l2: geometry collision mesh filename=package://walker_description/meshes/walker_head.dae; visual mesh filename=package://walker_description/meshes/walker_head.dae
- link head_l3: geometry 

Commit message: movement helpers quite working

File: ubt_sim_ws/src/walker_description/urdf/walker.urdf (robot description, URDF)
Before this commit: robot walker, 56 links, 55 joints
Links:
- added link left_tcp
- added link right_tcp
Joints:
- added joint left_tcp_joint: type fixed, parent left_palm_link, child left_tcp, origin xyz=-0.02 -0.05 0.015 rpy=0 0 -1.8, axis 0 0 0
- added joint right_tcp_joint: type fixed, parent right_palm_link, child right_tcp, origin xyz=0.02 -0.05 0.015 rpy=0 0 -1.34159265359, axis 0 0 0

Commit message: test step works

File: ubt_sim_ws/src/walker_description/urdf/walker.urdf (robot description, URDF)
Before this commit: robot walker, 58 links, 57 joints
Links:
- added link left_foot_sole
- added link right_foot_sole
Joints:
- added joint left_foot_sole: type fixed, parent left_leg_link2, child left_foot_sole, origin xyz=0 -0.064652 0 rpy=0 -1.5707 -1.5707, axis 0 0 0
- added joint right_foot_sole: type fixed, parent right_leg_link2, child right_foot_sole, origin xyz=0 -0.064652 0 rpy=0 -1.5707 -1.5707, axis 0 0 0

Commit message: init branch.

File: ubt_sim_ws/src/walker_description/urdf/walker.urdf (robot description, URDF)
Before this commit: robot walker, 60 links, 59 joints
Links:
- added link center_of_mass
Joints:
- added joint center_of_mass: type fixed, parent base_link, child center_of_mass, origin xyz=0 0 -0.26 rpy=0 0 -1.570795, axis 0 0 0

Commit message: it kinda walks backwards, veryslowly,  with pengin slide.

File: ubt_sim_ws/src/walker_description/urdf/walker.urdf (robot description, URDF)
Before this commit: robot walker, 61 links, 60 joints
Joints:
- joint center_of_mass: origin xyz=0 0 -0.26 rpy=0 0 -1.570795 -> xyz=0 0 -0.470128 rpy=0 0 -1.570795

Commit message: task 14 video

File: ubt_sim_ws/src/walker_description/urdf/walker.urdf (robot description, URDF)
Before this commit: robot walker, 61 links, 60 joints
Links:
- added link center_of_mass_with_box
Joints:
- added joint center_of_mass_with_box: type fixed, parent base_link, child center_of_mass_with_box, origin xyz=0.1 0 -0.570128 rpy=0 0 -1.570795, axis 0 0 0
